File: application_fpga.kicad_sch (KiCad schematic)
At the start: 35 parts, among them U6 ICE40UP5K-SG48ITR, U8 SST26VF080A-104I/SN

Commit message: Mise à jour du projet
Parts:
- added R4: 10k, Resistor_SMD:R_0805_2012Metric, symbol Device:R
- added SW1: SW_Push, Button_Switch_THT:SW_PUSH_6mm, symbol Switch:SW_Push
Connections:
- net +3.3V: now also SW1.1
- net GND: now also R4.2
- net TOUCH_EVENT: now also R4.1, SW1.2
Other:
- note added: "Touch button"

Commit message: Version sent to fabrication
Parts:
- removed R4: 10k, Resistor_SMD:R_0805_2012Metric, symbol Device:R
- removed SW1: SW_Push, Button_Switch_THT:SW_PUSH_6mm, symbol Switch:SW_Push
- removed U8: SST26VF080A-104I/SN, Package_SO:SOIC-8_3.9x4.9mm_P1.27mm, symbol mta1:W25Q80DVUXIE
- added SW2: PTS526_SK15_SMTR2_LFS, footprints:PTS526SK15SMTR2LFS, symbol PTS526_SK15_SMTR2_LFS:PTS526_SK15_SMTR2_LFS
- added U4: SST25VF080B-50-4x-S2Ax, Package_SO:SOIC-8_3.9x4.9mm_P1.27mm, symbol Memory_Flash:SST25VF080B-50-4x-S2Ax
- U6: footprint Package_DFN_QFN:QFN-48-1EP_7x7mm_P0.5mm_EP5.6x5.6mm -> Package_DFN_QFN:QFN-48-1EP_7x7mm_P0.5mm_EP5.3x5.3mm
Connections:
- net +3.3V: now also U4.8 (VDD)
- net APP_FLASH_HOLD: now also U6.13 (IOB_24a), U4.7 (~{HOLD})
- net APP_FLASH_WP: now also U6.12 (IOB_22b), U4.3 (~{WP})
- net APP_ICE_MISO: now also U4.2 (SO)
- net APP_ICE_MOSI: now also U4.5 (SI)
- net APP_ICE_SCK: now also U4.6 (SCK)
- net APP_ICE_SS: now also U4.1 (~{CE})
- net GND: now also SW2.1, SW2.2, U4.4 (VSS)
- net TOUCH_EVENT: now also SW2.3, SW2.4
- no-connect marks 23 -> 21
Other:
- moved on the sheet: C23, R23, R24, R25, R26
