File: powersupply.kicad_sch (KiCad schematic)
At the start: 19 parts, among them U1 MCP1824T-2502EOT, U2 NCV8164ASN120T1G, U9 NCP752BSN33T1G

Commit message: Version sent to fabrication
Parts:
- removed R1, R2, R22: 10k, Resistor_SMD:R_0805_2012Metric, symbol Device:R
Connections:
- net +1V2: now also U9.3 (EN)
- net +3.3V: now also C2.1, U1.1 (Vin), U1.3 (/SHDN)
- net +5V: now also U2.3 (EN); no longer C2.1, U1.1 (Vin)
- net SPI_VCC_OK: no longer names the net of U9.4 (PG)
- net SPI_VCC_OK: no longer U1.3 (/SHDN)
- net VCC_OK: no longer names the net of U2.4 (PG)
- net VCC_OK: no longer U9.3 (EN)
- no-connect marks 1 -> 3
Other:
- moved on the sheet: C1, C3
