File: tk1-0805copie.kicad_pcb (KiCad board)
At the start: 2 copper layers, 63 x 38.4 mm, 65 parts, among them P1 USB_C_Plug, U1 MCP1824T-2502EOT, U2 NCV8164ASN120T1G, U3 CH552E, U5 USBLC6-2SC6, U6 ICE40UP5K-SG48ITR, U8 W25Q80DVSNIG, U9 NCP752BSN33T1G

Commit message: Mise à jour du projet
Parts:
- added R4: 10k, Resistor_SMD:R_0805_2012Metric, F.Cu at (138.1, 86.8)
- added SW1: SW_Push, Button_Switch_THT:SW_PUSH_6mm, F.Cu at (137.0, 76.3)
- U8: value W25Q80DVSNIG -> SST26VF080A-104I/SN
- moved TP5 29.9 mm to (133.8, 76.0)
- moved TP4 26.2 mm to (96.1, 104.5)
- moved TP2 19.7 mm to (89.1, 104.5)
- moved TP1 19.6 mm to (85.8, 104.5)
- moved TP6 15.5 mm to (99.6, 104.5)
- moved TP28 13.3 mm to (82.7, 104.5)
- moved TP3 13.0 mm to (92.5, 104.5)
- moved TP21 12.6 mm to (117.4, 104.4)
- moved TP17 9.76 mm to (130.4, 76.0)
- moved TP16 9.48 mm to (123.1, 76.0)
- moved TP15 9.46 mm to (119.2, 76.0)
- moved TP7 9.40 mm to (103.0, 104.5)
- moved TP8 8.99 mm to (106.6, 104.5)
- moved TP9 8.55 mm to (110.1, 104.5)
- moved TP20 8.40 mm to (120.8, 104.4)
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Connections:
- U3 pad 6: INT_USB_D- -> INT_USB_D+
- U3 pad 7: INT_USB_D+ -> INT_USB_D-
- U5 pad 4: /USB to Serial converter/INT_USB_IN_D+ -> /USB to Serial converter/INT_USB_IN_D-
- U5 pad 6: /USB to Serial converter/INT_USB_IN_D- -> /USB to Serial converter/INT_USB_IN_D+
- U6 pad : (no net) -> APP_GPIO1
Routing:
- net GND: track 113.4 -> 48.9 mm, vias 22 -> 23
- net TOUCH_EVENT: track 0.00 -> 29.1 mm
- net +3.3V: track 90.3 -> 72.0 mm
- net +1V2: track 71.7 -> 89.3 mm
- net INTERFACE_TX: track 19.0 -> 33.5 mm
- net +2V5: track 34.3 -> 46.2 mm
- net APP_CDONE: track 12.4 -> 22.8 mm
- net APP_GPIO4: track 3.29 -> 13.1 mm
- net APP_ICE_SS: track 31.6 -> 40.3 mm
- net /Application FPGA/APP_FLASH_HOLD: track 44.7 -> 36.3 mm
- net APP_CRESET: track 12.7 -> 20.8 mm
- net INTERFACE_RX: track 24.1 -> 32.2 mm
- net INTERFACE_RTS: track 23.8 -> 31.4 mm
- net APP_GPIO1: track 10.7 -> 17.1 mm
- net APP_ICE_SCK: track 18.9 -> 23.9 mm
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Other:
- board size 63 x 38.4 mm -> 69.3 x 39.8 mm

Commit message: Version sent to fabrication
Parts:
- removed P1: USB_C_Plug, Connector_USB:USB_C_Receptacle_GCT_USB4085
- removed R1, R2, R22: 10k, Resistor_SMD:R_0805_2012Metric
- removed SW1: SW_Push, Button_Switch_THT:SW_PUSH_6mm
- removed U8: SST26VF080A-104I/SN, Package_SO:SOIC-8_3.9x4.9mm_P1.27mm
- added FB1: FerriteBead, Resistor_SMD:R_0805_2012Metric_Pad1.20x1.40mm_HandSolder, F.Cu at (83.0, 99.5)
- added J3: USB4085-GF-A_REVB, mta1:GCT_USB4085-GF-A_REVB, F.Cu at (80.2, 92.5)
- added SW2: PTS526_SK15_SMTR2_LFS, footprints:PTS526SK15SMTR2LFS, F.Cu at (131.5, 92.1)
- added TP14: APP_ICE_MOSI, mta1:TestPoint_Pad_D1.0mm, B.Cu at (120.9, 76.0)
- added U4: SST25VF080B-50-4x-S2Ax, Package_SO:SOIC-8_3.9x4.9mm_P1.27mm, F.Cu at (123.9, 79.2)
- R4: value 10k -> 5.1k; footprint Resistor_SMD:R_0805_2012Metric -> Resistor_SMD:R_0805_2012Metric_Pad1.20x1.40mm_HandSolder
- U6: footprint Package_DFN_QFN:QFN-48-1EP_7x7mm_P0.5mm_EP5.6x5.6mm -> Package_DFN_QFN:QFN-48-1EP_7x7mm_P0.5mm_EP5.3x5.3mm
- moved R4 50.7 mm to (87.4, 89.2), turned to -90 degrees
- moved FID1 32.6 mm to (81.2, 109.1)
- moved C23 26.8 mm to (123.7, 75.4), turned to 0 degrees
- moved TP5 24.1 mm to (109.8, 76.0)
- moved FID2 16.4 mm to (133.1, 110.2)
- moved C7 11.1 mm to (99.2, 96.2), turned to 0 degrees
- moved C2 10.8 mm to (91.5, 108.0)
- moved C13 10.1 mm to (99.2, 103.0), turned to 0 degrees
- moved TP16 8.87 mm to (131.9, 76.0)
- moved C4 8.34 mm to (99.4, 108.3)
- moved D3R1 7.29 mm to (129.9, 108.0)
- moved D3G1 7.03 mm to (130.0, 104.6)
- moved D3B1 6.98 mm to (130.0, 101.1)
- moved R20 5.85 mm to (128.1, 84.6)
- moved R18 5.28 mm to (125.6, 99.8)
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Connections:
- C16 pad 1: +1V2 -> VCC_OK
- C2 pad 1: +5V -> +3.3V
- C20 pad 1: +1V2 -> VCC_OK
- C5 pad 1: +1V2 -> VCC_OK
- FB3 pad 2: +1V2 -> VCC_OK
- R25 pad 2: /Application FPGA/APP_FLASH_WP -> APP_FLASH_WP
- R26 pad 2: /Application FPGA/APP_FLASH_HOLD -> APP_FLASH_HOLD
- R4 pad 1: TOUCH_EVENT -> Net-(J3-CC2)
- TP19 pad 1: /Application FPGA/APP_FLASH_WP -> APP_GPIO2
- TP20 pad 1: /Application FPGA/APP_FLASH_HOLD -> APP_GPIO3
- TP4 pad 1: +1V2 -> VCC_OK
- U1 pad 1: +5V -> +3.3V
- U1 pad 3: SPI_VCC_OK -> +3.3V
- U2 pad 3: Net-(U2-EN) -> +5V
- U2 pad 4: VCC_OK -> unconnected-(U2-PG-Pad4)
- U2 pad 5: +1V2 -> VCC_OK
- U5 pad 1: INT_USB_D+ -> INT_USB_D-
- U5 pad 3: INT_USB_D- -> INT_USB_D+
- U5 pad 4: /USB to Serial converter/INT_USB_IN_D- -> /USB to Serial converter/INT_USB_IN_D+
- U5 pad 6: /USB to Serial converter/INT_USB_IN_D+ -> /USB to Serial converter/INT_USB_IN_D-
- U6 pad : APP_GPIO1 -> (no net)
- U6 pad 12: unconnected-(U6-IOB_22b-Pad12) -> APP_FLASH_WP
- U6 pad 13: unconnected-(U6-IOB_24a-Pad13) -> APP_FLASH_HOLD
- U6 pad 30: +1V2 -> VCC_OK
- U6 pad 38: /Application FPGA/APP_FLASH_WP -> APP_GPIO2
- U6 pad 45: /Application FPGA/APP_FLASH_HOLD -> APP_GPIO3
- U6 pad 5: +1V2 -> VCC_OK
- U9 pad 4: SPI_VCC_OK -> unconnected-(U9-PG-Pad4)
Routing:
- net +1V2: track 89.3 -> 0.00 mm, vias 3 -> 0
- net VCC_OK: track 16.5 -> 85.3 mm, vias 0 -> 4
- net /Application FPGA/APP_FLASH_WP: track 39.6 -> 0.00 mm, vias 2 -> 0
- net +5V: track 39.7 -> 78.0 mm, vias 1 -> 5
- net /Application FPGA/APP_FLASH_HOLD: track 36.3 -> 0.00 mm, vias 2 -> 0
- net SPI_VCC_OK: track 33.2 -> 0.00 mm, vias 2 -> 0
- net GND: track 48.9 -> 70.7 mm, vias 23 -> 27
- net APP_FLASH_WP: track 0.00 -> 20.4 mm
- net APP_FLASH_HOLD: track 0.00 -> 19.2 mm, vias 0 -> 2
- net Net-(FB1-Pad1): track 0.00 -> 18.9 mm
- net TOUCH_EVENT: track 29.1 -> 15.5 mm
- net Net-(J3-CC2): track 0.00 -> 12.8 mm
- net +3.3V: track 72.0 -> 60.5 mm, vias 4 -> 3
- net APP_GPIO3: track 0.00 -> 10.6 mm, vias 0 -> 1
- net Net-(U2-EN): track 9.37 -> 0.00 mm
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Other:
- board size 69.3 x 39.8 mm -> 57.6 x 39.8 mm
- board text added: "+1.2V"
- board text added: "+2.5V"
- board text added: "+3.3V"
- board text added: "+5V"
- board text added: "11/03/2026"
- board text added: "CDONE"
- board text added: "CRESET"
- board text added: "CTS"
- board text added: "GND"
- board text added: "GPIO1"
- board text added: "GPIO2"
- board text added: "GPIO3"
- board text added: "GPIO4"
- board text added: "MISO"
- board text added: "MOSI"
- board text added: "RTS"
- board text added: "RX"
- board text added: "SCK"
- board text added: "SS"
- board text added: "TX"
