File: usb_to_serial.kicad_sch (KiCad schematic)
At the start: 10 parts, among them P1 USB_C_Plug, U3 CH552E, U5 USBLC6-2SC6

Commit message: Version sent to fabrication
Parts:
- removed P1: USB_C_Plug, Connector_USB:USB_C_Receptacle_GCT_USB4085, symbol Connector:USB_C_Plug
- added FB1: FerriteBead, Resistor_SMD:R_0805_2012Metric_Pad1.20x1.40mm_HandSolder, symbol Device:FerriteBead
- added J3: USB4085-GF-A_REVB, mta1:GCT_USB4085-GF-A_REVB, symbol USB4085-GF-A_REVB:USB4085-GF-A_REVB
- added R4: 5.1k, Resistor_SMD:R_0805_2012Metric_Pad1.20x1.40mm_HandSolder, symbol Device:R
Connections:
- net +5V: now also J3.A4 (VBUS), J3.A9 (VBUS), J3.B4 (VBUS), J3.B9 (VBUS)
- net GND: now also FB1.2, J3.A1 (GND), J3.A12 (GND), J3.B1 (GND), J3.B12 (GND), R4.2
- net INT_USB_D+: now also U5.3 (I/O2); no longer U5.1 (I/O1)
- net INT_USB_D-: now also U5.1 (I/O1); no longer U5.3 (I/O2)
- net INT_USB_IN_D+: now also U5.4 (I/O2), J3.A6 (DP1), J3.B6 (DP2); no longer U5.6 (I/O1)
- net INT_USB_IN_D-: now also U5.6 (I/O1), J3.A7 (DN1), J3.B7 (DN2); no longer U5.4 (I/O2)
- net at R29.1: now also J3.A5 (CC1)
- new net: FB1.1, J3.S1 (SHELL), J3.S2 (SHELL), J3.S3 (SHELL), J3.S4 (SHELL)
- new net: J3.B5 (CC2), R4.1
- no-connect marks 12 -> 3
